File: keyboard_pcb/keyboard_pcb.kicad_pcb (KiCad board)
At the start: 2 copper layers, 347.7 x 119.1 mm, 190 parts, among them SW1 ESC, SW10 F9, SW11 F10, SW12 F11, SW13 F12, SW14 PRNTSC, SW15 SCRLLK, SW16 PBRK, SW17 `, SW18 #1, SW19 #2, SW2 F1, SW20 #3, SW21 #4, SW22 #5, SW23 #6, SW24 #7, SW25 #8, SW26 #9, SW27 #0, SW28 -, SW29 =, SW3 F2, SW30 BKSPC, SW31 INS, SW32 HOME, SW33 PGUP, SW34 TAB, SW35 Q, SW36 W, SW37 E, SW38 R, SW39 T, SW4 F3, SW40 Y, SW41 U, SW42 I, SW43 O, SW44 P, SW45 [, SW46 ], SW47 \, SW48 DEL, SW49 END, SW5 F4, SW50 PGDN, SW51 CAPSLK, SW52 A, SW53 S, SW54 D, SW55 F, SW56 G, SW57 H, SW58 J, SW59 K, SW6 F5, SW60 L, SW61 ;, SW62 ', SW63 ENTER, SW64 LSHIFT, SW65 Z, SW66 X, SW67 C, SW68 V, SW69 B, SW7 F6, SW70 N, SW71 M, SW72 ,, SW73 ., SW74 /, SW75 RSHIFT, SW76 UP, SW77 LCTRL, SW78 LWIN, SW79 LALT, SW8 F7, SW80 SPACE, SW81 RALT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

Commit message: TKL Prototype V1.0
Routing:
- added copper zone on B.Cu, net GND
Other:
- board text added: "TKL Prototype V1.0"
Changed lines of the file:
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@@
 		(layer "Edge.Cuts")
 	)
+	(gr_text "TKL Prototype V1.0"
+		(at 134.14375 196.05625 0)
+		(layer "F.SilkS")
+		(effects
+			(font
+				(size 1 1)
+				(thickness 0.1)
+			)
+			(justify left bottom)
+		)
+	)
 	(segment
 		(start 200.4625 202.5)
@@
 		(net 122)
 	)
+	(zone
+		(net 2)
+		(net_name "GND")
+		(layer "B.Cu")
+		(hatch edge 0.5)
+		(priority 1)
+		(connect_pads
+			(clearance 0.5)
+		)
+		(min_thickness 0.25)
+		(filled_areas_thickness no)
+		(fill yes
+			(thermal_gap 0.5)
+			(thermal_bridge_width 0.5)
+		)
+		(polygon
+			(pts
+				(xy 234 88.5) (xy 245.5 88.5) (xy 245.5 104) (xy 234 104)
+			)
+		)
+	)
+	(zone
+		(net 2)
+		(net_name "GND")
+		(layer "B.Cu")
+		(hatch edge 0.5)
+		(connect_pads
+			(clearance 0.5)
+		)
+		(min_thickness 0.25)
+		(filled_areas_thickness no)
+		(fill yes
+			(thermal_gap 0.5)
+			(thermal_bridge_width 0.5)
+		)
+		(polygon
+			(pts
+				(xy 212 183) (xy 212 204.5) (xy 178 204.5) (xy 178 183)
+			)
+		)
+	)
 )
